File: LtStagger/LTStagger_Bottom_Corners.kicad_pcb (KiCad board)
At the start: 2 copper layers, 42.5 x 41 mm, 3 parts

Commit message: about to give an angle and dog bones
Parts:
- removed the REF** at (55.8, 91.7)
- removed the REF** at (59.0, 94.8)
- added G***: LOGO, Digi:PieCn, B.Cu at (85.0, 66.5)
- added REF**: breakaway-mousebites, Keebio-Parts:breakaway-mousebites, F.Cu at (93.6, 91.5)
- added REF**: breakaway-mousebites, Keebio-Parts:breakaway-mousebites, F.Cu at (84.3, 82.5)
- added REF**: Long_Pad_single_sided, Digi:Long_Pad_single_sided, F.Cu at (97.0, 58.0)
- added REF**: Long_Pad_single_sided, Digi:Long_Pad_single_sided, F.Cu at (94.3, 55.3)
- added REF**: breakaway-mousebites, Keebio-Parts:breakaway-mousebites, F.Cu at (69.0, 67.1)
- added REF**: breakaway-mousebites, Keebio-Parts:breakaway-mousebites, F.Cu at (59.7, 58.1)
- added REF**: Long_Pad_single_sided, Digi:Long_Pad_single_sided, F.Cu at (56.4, 91.7)
- added REF**: Long_Pad_single_sided, Digi:Long_Pad_single_sided, F.Cu at (59.0, 94.3)
- G***: moved to B.Cu
- moved G*** 1.58 mm to (68.7, 83.0), turned to 180 degrees
Other:
- board size 42.5 x 41 mm -> 45 x 43.3 mm
