File: LtStagger/LTStagger_Left_Right_side.kicad_pcb (KiCad board)
At the start: 2 copper layers, 112 x 30 mm, 5 parts

Commit message: about to give an angle and dog bones
Parts:
- removed the REF** at (121.7, 160.4)
- removed the REF** at (-24.4, 140.3)
- removed the REF** at (16.4, 137.2)
- removed the REF** at (125.2, 137.6)
- removed the REF** at (-24.8, 133.6)
- added REF**: Long_Pad_single_sided, Digi:Long_Pad_single_sided, F.Cu at (171.2, 66.4)
- added REF**: Long_Pad_single_sided, Digi:Long_Pad_single_sided, F.Cu at (25.1, 47.5)
- added REF**: Long_Pad_single_sided, Digi:Long_Pad_single_sided, F.Cu at (66.4, 43.8)
- added REF**: Long_Pad_single_sided, Digi:Long_Pad_single_sided, F.Cu at (174.1, 44.2)
- added REF**: Long_Pad_single_sided, Digi:Long_Pad_single_sided, F.Cu at (24.7, 40.8)
