File: LtStagger/LTStagger_back_side.kicad_pcb (KiCad board)
At the start: 2 copper layers, 155 x 30 mm, 4 parts

Commit message: about to give an angle and dog bones
Parts:
- removed the REF** at (132.7, 160.4)
- removed the REF** at (129.2, 137.6)
- removed the REF** at (277.8, 140.2)
- added REF**: Long_Pad_single_sided, Digi:Long_Pad_single_sided, F.Cu at (202.1, 36.7)
- added REF**: Long_Pad_single_sided, Digi:Long_Pad_single_sided, F.Cu at (54.5, 59.1)
- added REF**: Long_Pad_single_sided, Digi:Long_Pad_single_sided, F.Cu at (51.5, 36.9)
- added REF**: Long_Pad_single_sided, Digi:Long_Pad_single_sided, F.Cu at (199.6, 40.1)
- moved REF** 127.1 mm to (199.6, 33.5)
