File: LtStagger/LTStagger_sides.kicad_pcb (KiCad board)
At the start: 2 copper layers, 267.8 x 106.5 mm, 12 parts

Commit message: about to give an angle and dog bones
Parts:
- removed the REF** at (55.8, 91.7)
- removed the REF** at (277.8, 140.2)
- removed the REF** at (59.0, 94.8)
- removed the REF** at (121.7, 160.4)
- removed the REF** at (132.7, 160.4)
- removed the REF** at (-24.4, 140.3)
- removed the REF** at (16.4, 137.2)
- removed the REF** at (125.2, 137.6)
- removed the REF** at (-24.8, 133.6)
- removed the REF** at (129.2, 137.6)
- added REF**: Long_Pad_single_sided, Digi:Long_Pad_single_sided, F.Cu at (280.2, 137.4)
- added REF**: Long_Pad_single_sided, Digi:Long_Pad_single_sided, F.Cu at (129.7, 137.6)
- added REF**: Long_Pad_single_sided, Digi:Long_Pad_single_sided, F.Cu at (277.8, 140.8)
- added REF**: Long_Pad_single_sided, Digi:Long_Pad_single_sided, F.Cu at (56.4, 91.7)
- added REF**: Long_Pad_single_sided, Digi:Long_Pad_single_sided, F.Cu at (59.0, 94.3)
- added REF**: Long_Pad_single_sided, Digi:Long_Pad_single_sided, F.Cu at (121.7, 159.8)
- added REF**: Long_Pad_single_sided, Digi:Long_Pad_single_sided, F.Cu at (132.7, 159.8)
- added REF**: Long_Pad_single_sided, Digi:Long_Pad_single_sided, F.Cu at (-24.4, 140.8)
- added REF**: Long_Pad_single_sided, Digi:Long_Pad_single_sided, F.Cu at (16.9, 137.2)
- added REF**: Long_Pad_single_sided, Digi:Long_Pad_single_sided, F.Cu at (124.6, 137.6)
- added REF**: Long_Pad_single_sided, Digi:Long_Pad_single_sided, F.Cu at (-24.8, 134.2)
- moved REF** 0.43 mm to (277.8, 134.2)
Changed lines of the file:
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@@
     (tracks 0)
     (zones 0)
-    (modules 12)
+    (modules 13)
     (nets 1)
   )
@@
   )
   (module Digi:Long_Pad_single_sided (layer F.Cu)
-    (at 55.8 91.65 90)
+    (at 280.25 137.4 270)
+    (fp_text reference REF** (at 0 0.5 90) (layer F.SilkS)
+      (effects (font (size 1 1) (thickness 0.15)))
+    )
+    (fp_text value Long_Pad_single_sided (at 0 -0.5 90) (layer F.Fab)
+      (effects (font (size 1 1) (thickness 0.15)))
+    )
+    (pad 1 smd oval (at 146.05 0 270) (size 5 1) (layers F.Cu F.Paste F.Mask))
+    (pad 1 smd oval (at 139.7 0 270) (size 5 1) (layers F.Cu F.Paste F.Mask))
+    (pad 1 smd oval (at 133.35 0 270) (size 5 1) (layers F.Cu F.Paste F.Mask))
+    (pad 1 smd oval (at 127 0 270) (size 5 1) (layers F.Cu F.Paste F.Mask))
+    (pad 1 smd oval (at 120.65 0 270) (size 5 1) (layers F.Cu F.Paste F.Mask))
+    (pad 1 smd oval (at 114.3 0 270) (size 5 1) (layers F.Cu F.Paste F.Mask))
+    (pad 1 smd oval (at 107.95 0 270) (size 5 1) (layers F.Cu F.Paste F.Mask))
+    (pad 1 smd oval (at 101.6 0 270) (size 5 1) (layers F.Cu F.Paste F.Mask))
+    (pad 1 smd oval (at 95.25 0 270) (size 5 1) (layers F.Cu F.Paste F.Mask))
+    (pad 1 smd oval (at 88.9 0 270) (size 5 1) (layers F.Cu F.Paste F.Mask))
+    (pad 1 smd oval (at 82.55 0 270) (size 5 1) (layers F.Cu F.Paste F.Mask))
+    (pad 1 smd oval (at 76.2 0 270) (size 5 1) (layers F.Cu F.Paste F.Mask))
+    (pad 1 smd oval (at 69.85 0 270) (size 5 1) (layers F.Cu F.Paste F.Mask))
+    (pad 1 smd oval (at 63.5 0 270) (size 5 1) (layers F.Cu F.Paste F.Mask))
+    (pad 1 smd oval (at 57.15 0 270) (size 5 1) (layers F.Cu F.Paste F.Mask))
+    (pad 1 smd oval (at 50.8 0 270) (size 5 1) (layers F.Cu F.Paste F.Mask))
+    (pad 1 smd oval (at 44.45 0 270) (size 5 1) (layers F.Cu F.Paste F.Mask))
+    (pad 1 smd oval (at 38.1 0 270) (size 5 1) (layers F.Cu F.Paste F.Mask))
+    (pad 1 smd oval (at 31.75 0 270) (size 5 1) (layers F.Cu F.Paste F.Mask))
+    (pad 1 smd oval (at 25.4 0 270) (size 5 1) (layers F.Cu F.Paste F.Mask))
+    (pad 1 smd oval (at 19.05 0 270) (size 5 1) (layers F.Cu F.Paste F.Mask))
+    (pad 1 smd oval (at 12.7 0 270) (size 5 1) (layers F.Cu F.Paste F.Mask))
+    (pad 1 smd oval (at 6.35 0 270) (size 5 1) (layers F.Cu F.Paste F.Mask))
+    (pad 1 smd oval (at 0 0 270) (size 5 1) (layers F.Cu F.Paste F.Mask))
+  )
+  (module Digi:Long_Pad_single_sided (layer F.Cu)
+    (at 56.35 91.65 90)
     (fp_text reference REF** (at 0 0.5 90) (layer F.SilkS)
       (effects (font (size 1 1) (thickness 0.15)))
@@
   )
   (module Digi:Long_Pad_single_sided (layer F.Cu)
-    (at 59 94.85)
+    (at 58.95 94.3)
     (fp_text reference REF** (at 0 0.5) (layer F.SilkS)
       (effects (font (size 1 1) (thickness 0.15)))
@@
   )
   (module Digi:Long_Pad_single_sided (layer F.Cu)
-    (at 121.675 160.375 180)
+    (at 121.7 159.8 180)
     (fp_text reference REF** (at 0 0.5) (layer F.SilkS)
       (effects (font (size 1 1) (thickness 0.15)))
@@
   )
   (module Digi:Long_Pad_single_sided (layer F.Cu)
-    (at 132.725 160.4)
+    (at 132.7 159.8)
     (fp_text reference REF** (at 0 0.5) (layer F.SilkS)
       (effects (font (size 1 1) (thickness 0.15)))
@@
   )
   (module Digi:Long_Pad_single_sided (layer F.Cu)
-    (at -24.375 140.275)
+    (at -24.375 140.85)
     (fp_text reference REF** (at 0 0.5) (layer F.SilkS)
       (effects (font (size 1 1) (thickness 0.15)))
@@
   )
   (module Digi:Long_Pad_single_sided (layer F.Cu)
-    (at 16.4 137.175 270)
+    (at 16.95 137.175 270)
     (fp_text reference REF** (at 0 0.5 90) (layer F.SilkS)
       (effects (font (size 1 1) (thickness 0.15)))
@@
   )
   (module Digi:Long_Pad_single_sided (layer F.Cu)
-    (at 125.2 137.6 270)
+    (at 124.6 137.6 270)
     (fp_text reference REF** (at 0 0.5 90) (layer F.SilkS)
       (effects (font (size 1 1) (thickness 0.15)))
@@
   )
   (module Digi:Long_Pad_single_sided (layer F.Cu)
-    (at -24.75 133.625)
+    (at -24.75 134.15)
     (fp_text reference REF** (at 0 0.5) (layer F.SilkS)
       (effects (font (size 1 1) (thickness 0.15)))
@@
   )
   (module Digi:Long_Pad_single_sided (layer F.Cu)
-    (at 129.15 137.575 270)
+    (at 129.7 137.55 270)
     (fp_text reference REF** (at 0 0.5 90) (layer F.SilkS)
       (effects (font (size 1 1) (thickness 0.15)))
@@
   )
   (module Digi:Long_Pad_single_sided (layer F.Cu)
-    (at 277.775 140.25 180)
+    (at 277.775 140.85 180)
     (fp_text reference REF** (at 0 0.5) (layer F.SilkS)
       (effects (font (size 1 1) (thickness 0.15)))
@@
   )
   (module Digi:Long_Pad_single_sided (layer F.Cu)
-    (at 277.725 133.725 180)
-    (fp_text reference REF** (at 0 0.5) (layer F.SilkS)
-      (effects (font (size 1 1) (thickness 0.15)))
+    (at 277.75 134.15 180)
+    (fp_text reference REF** (at 0 0.5) (layer F.SilkS)
+      (effects (font (size 1 1) (thickness 0.15)))

Commit message: Maybe ready for production
Parts:
- removed G***: LOGO, Digi:PieCn
- removed REF** (x12): Long_Pad_single_sided, Digi:Long_Pad_single_sided
- added ?: , Digi:Right, B.Cu at (160.9, 104.6)
- added ?: , Digi:Left, B.Cu at (115.3, 104.6)
- added ?: , Digi:Right, B.Cu at (161.0, 46.7)
- added ?: , Digi:Left, B.Cu at (128.5, 47.0)
Other:
- board size 267.8 x 106.5 mm -> 227 x 87.1 mm
- board text added: "Left Keyboard"
- board text added: "Left Side"
- board text added: "Right Keyboard"
- board text added: "Right Side"
