File: LtStagger/dimensions.kicad_pcb (KiCad board)
At the start: 2 copper layers, 151.4 x 105.6 mm, 51 parts, among them K0 K00, K1 K01, K10 K10, K11 K11, K12 K12, K2 K02, K20 K20, K21 K21, K22 K22, K30 K30, K31 K31, K32 K32, K33 K33, K40 K40, K41 K41, K42 K42, K43 K43, K50 K50, K51 K51, K53 K53, SW1 Rotary_Encoder_Switch, U1 ProMicro, U2 TRRS, U3 MCP23018-E_SP

Commit message: Ready for first review
Routing:
- net Row1: track 214.8 -> 0.00 mm
- net Row2: track 197.3 -> 0.00 mm
- net Row0: track 197.2 -> 0.00 mm
- net GND: track 193.4 -> 0.00 mm
- net Row3: track 192.0 -> 0.00 mm
- net Col3: track 190.4 -> 0.00 mm
- net Col4: track 190.1 -> 0.00 mm
- net Col2: track 171.8 -> 0.00 mm
- net VCC: track 167.3 -> 0.00 mm
- net Col0: track 160.5 -> 0.00 mm
- net SDA: track 147.3 -> 0.00 mm
- net SCL: track 145.7 -> 0.00 mm
- net Col1: track 143.4 -> 0.00 mm
- net Col5: track 129.7 -> 0.00 mm
- net Net-(D51-Pad2): track 20.7 -> 0.00 mm
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
Commit message: dog bones and curve
Other:
- board size 151.4 x 105.6 mm -> 440.7 x 157.5 mm

Commit message: Maybe ready for production
Parts:
- added ?: , Digi:Left, F.Cu at (314.2, 149.8)
- added ?: , Digi:Right, B.Cu at (314.2, 149.8)
- added ?: , Digi:Right, B.Cu at (356.3, 6.06)
- added ?: , Digi:Left, B.Cu at (310.7, 6.05)
- added ?: , Digi:Right, B.Cu at (125.0, 4.18)
- added ?: , Digi:Left, B.Cu at (92.5, 4.47)
- added G***: LOGO, Digi:PieCn, F.Cu at (276.1, 69.2)
- added G***: LOGO, Digi:PieCn, B.Cu at (276.4, 69.2)
Other:
- board size 440.7 x 157.5 mm -> 456.3 x 245.3 mm
- board text added: "Left Keyboard"
- board text added: "Left Side"
- board text added: "Right Keyboard"
- board text added: "Right Side"
