File: LtStagger/LTStagger_ALL.kicad_pcb (KiCad board)
At the start: 2 copper layers, 430.3 x 180.8 mm, 120 parts, among them K0 K00, K1 K01, K10 K10, K11 K11, K12 K12, K2 K02, K20 K20, K21 K21, K22 K22, K30 K30, K31 K31, K32 K32, K33 K33, K40 K40, K41 K41, K42 K42, K43 K43, K50 K50, K51 K51, K53 K53, SW1 Rotary_Encoder_Switch, U1 ProMicro, U2 TRRS, U3 MCP23018-E_SP

Commit message: Unknown status, but this is how I found it today.
Parts:
- added REF**: , Digi:Mounting Holes, F.Cu at (78.3, 141.2)
- added REF**: SW_PUSH, Keebio-Parts:SW_Tactile_SPST_Angled_MJTP1117, F.Cu at (396.2, 199.6)
- added REF**: , Digi:Long_Pad_single_sided_2, F.Cu at (244.1, 166.2)
- added REF**: , Digi:Long_Pad_single_sided_2, F.Cu at (332.1, 166.1)
- added REF**: , Digi:Long_Pad_single_sided_2, F.Cu at (332.3, 133.8)
- added REF**: , Digi:Long_Pad_single_sided_2, F.Cu at (244.3, 133.8)
- added REF**: , Digi:Long_Pad_single_sided_2, F.Cu at (483.3, 237.9)
- added REF**: , Digi:Long_Pad_single_sided_2, F.Cu at (395.3, 237.9)
- added REF**: , Digi:Long_Pad_single_sided_2, F.Cu at (392.6, 270.2)
- added REF**: , Digi:Long_Pad_single_sided_2, F.Cu at (480.6, 270.2)
- REF** (x6): value Long_Pad_single_sided_1 -> (none)
- REF** (x10): value Long_Pad_single_sided_3tight -> (none)
- REF** (x4): value Long_Pad_single_sided_2 -> (none)
- REF** (x4): value Long_Pad_single_sided_3 -> (none)
- REF** (x4): value Long_Pad_single_sided_shorter -> (none)
- REF** (x2): value Long_Pad_single_sided -> (none)
- REF** (x2): value Long_Pad_double_sided_shorter -> (none)
- REF** (x2): value Long_Pad_double_sided -> (none)
- REF**: value Mounting Holes -> (none)
- SW1: footprint Keebio-Parts:RotaryEncoder_EC11 -> Digi:RotaryEncoder_EC11_plate
Routing:
- net (no net): track 2961.0 -> 3161.8 mm
Other:
- outline, holes or cut-outs redrawn
- board text added: "LTStagger - Alpha1 ©2020 LovesTha"
