File: LtStagger2/LTStagger.kicad_sch (KiCad schematic)
At the start: 48 parts, among them K0 K00, K1 K01, K10 K10, K11 K11, K12 K12, K2 K02, K20 K20, K21 K21, K22 K22, K30 K30, K31 K31, K32 K32, K40 K40, K41 K41, K42 K42, K50 K50, K51 K51, K60 K50, K61 K51, SW2 SW_Push_45deg, U2 TRRS, U3 Pico, U5 COM-09032

Commit message: Time to test footprints
Parts:
- added H1, H2, H3, H4: MountingHole, MountingHole:MountingHole_4.3mm_M4_ISO7380_Pad_TopBottom, symbol Mechanical:MountingHole
- added H5: MountingHole, misc:trackball-mount, symbol Mechanical:MountingHole
- added J-RGB1: Conn_01x03, Connector:FanPinHeader_1x03_P2.54mm_Vertical, symbol Connector_Generic:Conn_01x03
- added J1: Conn_02x07_Odd_Even, Connector_PinHeader_2.54mm:PinHeader_2x07_P2.54mm_Vertical, symbol Connector_Generic:Conn_02x07_Odd_Even
- added JC1: MountingHole, symbol Mechanical:MountingHole
- added R1: 500R, Resistor_SMD:R_0805_2012Metric_Pad1.20x1.40mm_HandSolder, symbol Device:R
- added U1: ~, misc:joycon-thumbstick-with-ZIF, symbol Misc:JoyConStick
- K0, K1, K10, K11, K12, K2, K20, K21, K22, K30, K31, K32, K40, K41, K42: footprint Button_Switch_Keyboard:SW_Cherry_MX_1.00u_PCB -> misc:SW_Cherry_MX_1.00u_PCB_with_4960; symbol Switch:SW_Push -> Misc:4960-with-switch
- K50, K51, K60, K61: footprint misc:Low-Profile-Choc-MX -> misc:Low-Profile-Choc-MX-with-4960-LED; symbol Switch:SW_Push -> Misc:4960-with-switch
- U3: footprint misc:RPi_Pico_SMD_TH_reduced -> misc:RPi_Pico_SMD_TH_reduced_extra
- renumbered D0 to D00, D1 to D01, D2 to D02, R4 to R2, R5 to R3
Connections:
- net +3.3V: now also J1.1 (Pin_1), U1.5 (3.3V)
- net Axis1: now also U1.4 (Axis1)
- net Axis2: now also U1.1 (Axis2)
- net Col0: now also J1.14 (Pin_14)
- net Col1: now also J1.13 (Pin_13)
- net Col2: now also J1.12 (Pin_12)
- net Col3: now also J1.11 (Pin_11)
- net Col4: now also J1.10 (Pin_10)
- net Col5: now also J1.9 (Pin_9)
- net GND: now also K0.5 (GND), K1.5 (GND), K10.5 (GND), K11.5 (GND), K12.5 (GND), K2.5 (GND), K20.5 (GND), K21.5 (GND), K22.5 (GND), K30.5 (GND), K31.5 (GND), K32.5 (GND), K40.5 (GND), K41.5 (GND), K42.5 (GND), K50.5 (GND), K51.5 (GND), K60.5 (GND), K61.5 (GND), J-RGB1.3 (Pin_3), J1.2 (Pin_2), U1.2 (GND)
- net VCC: now also K0.3 (VDD), K1.3 (VDD), K10.3 (VDD), K11.3 (VDD), K12.3 (VDD), K2.3 (VDD), K20.3 (VDD), K21.3 (VDD), K22.3 (VDD), K30.3 (VDD), K31.3 (VDD), K32.3 (VDD), K40.3 (VDD), K41.3 (VDD), K42.3 (VDD), K50.3 (VDD), K51.3 (VDD), K60.3 (VDD), K61.3 (VDD), J-RGB1.1 (Pin_1)
- net MISO: now reaches U3.1 (GPIO0)
- net MISO: now also J1.5 (Pin_5)
- net RGB: now reaches U3.11 (GPIO8)
- net RGB: now also R1.1
- net SPICS: now reaches U3.2 (GPIO1)
- net SPICS: now also J1.4 (Pin_4)
- net Row3: now reaches U3.25 (GPIO19)
- net Row3: now also J1.8 (Pin_8)
- net JoyButtonDirect: now reaches U3.29 (GPIO22)
- net JoyButtonDirect: now also U1.3 (Button)
- net Row4: now reaches U3.34 (GPIO28_ADC2)
- net Row4: now also J1.7 (Pin_7)
- net SCLK: now reaches U3.4 (GPIO2)
- net SCLK: now also J1.3 (Pin_3)
- net MOSI: now reaches U3.5 (GPIO3)
- net MOSI: now also J1.6 (Pin_6)
- new net: K2.4 (DOUT), K41.6 (DIN)
- new net: K12.4 (DOUT), K2.6 (DIN)
- new net: K1.4 (DOUT), K40.6 (DIN)
- new net: K1.6 (DIN), K11.4 (DOUT)
- new net: K0.6 (DIN), K10.4 (DOUT)
- new net: K12.6 (DIN), K22.4 (DOUT)
- new net: K11.6 (DIN), K21.4 (DOUT)
- new net: K10.6 (DIN), K20.4 (DOUT)
- new net: K22.6 (DIN), K32.4 (DOUT)
- new net: K21.6 (DIN), K31.4 (DOUT)
- new net: K20.6 (DIN), K30.4 (DOUT)
- new net: K32.6 (DIN), K42.4 (DOUT)
- new net: K31.6 (DIN), K41.4 (DOUT)
- new net: K30.6 (DIN), K40.4 (DOUT)
- new net: K42.6 (DIN), K61.4 (DOUT)
- new net: K51.4 (DOUT), K60.6 (DIN)
- new net: K50.4 (DOUT), K51.6 (DIN)
- new net: K50.6 (DIN), R1.2
- new net: K60.4 (DOUT), K61.6 (DIN)
- new net RGB-EXT: J-RGB1.2 (Pin_2), K0.4 (DOUT)
Other:
- moved on the sheet: R2, R3, SW2, U2, U3, U5

Commit message: Libraries
Parts:
- added R10, R11, R12, R4, R5, R6, R7, R8, R9: R, Resistor_SMD:R_0805_2012Metric_Pad1.20x1.40mm_HandSolder, symbol Device:R
- added S1, S2, S3, S4: NeoPixel_THT, LED_SMD:LED_WS2812B-Mini_PLCC4_3.5x3.5mm, symbol LED:NeoPixel_THT
Connections:
- net GND: now also S1.2 (GND), S2.2 (GND), S3.2 (GND), S4.2 (GND)
- net RGB: now also R4.2, R5.2, R6.2; no longer U3.11 (GPIO8)
- net VCC: now also S1.3 (VDD), S2.3 (VDD), S3.3 (VDD), S4.3 (VDD)
- net at R1.2: now also U3.11 (GPIO8); no longer K50.6 (DIN)
- net RGB-EXT renamed RGB-Ext-In
- net RGB-Ext-In: now also R10.1, R4.1, R7.1; no longer K0.4 (DOUT)
- new net: S3.1 (DOUT), S4.4 (DIN)
- new net: S2.1 (DOUT), S3.4 (DIN)
- new net: S1.1 (DOUT), S2.4 (DIN)
- new net RGB-MAT-IN: K50.6 (DIN), R12.1, R6.1, R9.1
- new net RGB-MAT-OUT: K0.4 (DOUT), R7.2, R8.2, R9.2
- new net RGB-Status-In: R11.1, R5.1, R8.1, S1.4 (DIN)
- new net RGB-Status-Out: R10.2, R11.2, R12.2, S4.1 (DOUT)
